Commit message: fix name: wheel_left-> wheel_l, wheel_right->wheel_r

File: kobuki_description/urdf/kobuki.urdf.xacro (robot description, xacro)
@@ -56,11 +56,11 @@
       </inertial>
     </link>
-    <joint name="wheel_left_joint" type="continuous">
-      <parent link="base_link"/>
-      <child link="wheel_left_link"/>
+    <joint name="wheel_l_joint" type="continuous">
+      <parent link="base_link"/>
+      <child link="wheel_l_link"/>
       <origin xyz="0.00 ${0.23/2} 0.0250" rpy="${-M_PI/2} 0 0"/>
       <axis xyz="0 0 1"/>
     </joint>
-    <link name="wheel_left_link">
+    <link name="wheel_l_link">
       <visual>
         <geometry>
@@ -83,11 +83,11 @@
       </inertial>
     </link>
-    <joint name="wheel_right_joint" type="continuous">
-      <parent link="base_link"/>
-      <child link="wheel_right_link"/>
+    <joint name="wheel_r_joint" type="continuous">
+      <parent link="base_link"/>
+      <child link="wheel_r_link"/>
       <origin xyz="0.00 -${0.23/2} 0.0250" rpy="${-M_PI/2} 0 0"/>
       <axis xyz="0 0 1"/>
     </joint>
-    <link name="wheel_right_link">
+    <link name="wheel_r_link">
       <visual>
         <geometry>

File: kobuki_description/urdf/kobuki_gazebo.urdf.xacro (robot description, xacro)
@@ -2,5 +2,5 @@
 <robot name="kobuki_sim" xmlns:xacro="http://ros.org/wiki/xacro">
   <xacro:macro name="kobuki_sim">
-    <gazebo reference="wheel_left_link">
+    <gazebo reference="wheel_l_link">
       <mu1>1.0</mu1>
       <mu2>1.0</mu2>
@@ -10,5 +10,5 @@
       <maxVel>1.0</maxVel>
     </gazebo>
-    <gazebo reference="wheel_right_link">
+    <gazebo reference="wheel_r_link">
       <mu1>1.0</mu1>
       <mu2>1.0</mu2>
@@ -163,6 +163,6 @@
       <plugin name="kobuki_controller" filename="libgazebo_ros_kobuki.so">
         <publish_tf>1</publish_tf>
-        <left_wheel_joint_name>wheel_left_joint</left_wheel_joint_name>
-        <right_wheel_joint_name>wheel_right_joint</right_wheel_joint_name>
+        <left_wheel_joint_name>wheel_l_joint</left_wheel_joint_name>
+        <right_wheel_joint_name>wheel_r_joint</right_wheel_joint_name>
         <wheel_separation>.230</wheel_separation>
         <wheel_diameter>0.070</wheel_diameter>
